File: PCB/environmental-monitor-pcb/environmental-monitor-pcb.kicad_pcb (KiCad board)
At the start: 2 copper layers, 64.5 x 82 mm, 4 parts, among them J2 ESP32 RIGHT HEADER, J3 BME280 MODULE, J4 SSD1306 OLED

Commit message: Add microSD card to environmental monitor PCB
Parts:
- added J5: Conn_01x06, Connector_PinHeader_2.54mm:PinHeader_1x06_P2.54mm_Vertical, F.Cu at (113.8, 77.8)
Connections:
- 3V3 pad 10: unconnected-(3V3-Pin_10-Pad10) -> /MISO
- 3V3 pad 14: unconnected-(3V3-Pin_14-Pad14) -> /SCL
- 3V3 pad 15: /SCL -> /MOSI
- 3V3 pad 8: unconnected-(3V3-Pin_8-Pad8) -> /CS
- 3V3 pad 9: unconnected-(3V3-Pin_9-Pad9) -> /SCK
Routing:
- net /MOSI: track 0.00 -> 59.7 mm
- net /CS: track 0.00 -> 55.9 mm
- net /SCK: track 0.00 -> 46.7 mm
- net /MISO: track 0.00 -> 44.1 mm
- net GND: track 114.4 -> 133.2 mm
- net +3V3: track 108.0 -> 126.8 mm
- net /SCL: track 51.5 -> 52.5 mm
Other:
- board size 64.5 x 82 mm -> 63.5 x 95.5 mm
